File: PCB_files/Sprinkler_Controller_V2/Sprinkler_Controller_V2/Sprinkler_Controller_V2.kicad_pcb (KiCad board)
At the start: 2 copper layers, 116 x 72 mm, 43 parts, among them J1 Screw_Terminal_01x02, J2 Screw_Terminal_01x11, SW1 SW_SPST, U1 ESP32_DevKit_V1_DOIT, U12 TPP362081-T6TR

Commit message: changed C1,C2 capacitor values
Parts:
- C1, C2: value 2200uF -> 1000uF
Changed lines of the file:
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@@
 			)
 		)
-		(property "Value" "2200uF"
+		(property "Value" "1000uF"
 			(at 0.112755 3.6 90)
 			(layer "F.Fab")
@@
 			)
 		)
-		(property "Value" "2200uF"
+		(property "Value" "1000uF"
 			(at 3.75 9.25 90)
 			(layer "F.Fab")
@@
 			(pts
 				(xy 144 104.2) (xy 144 102) (xy 144.8 100.2) (xy 144.8 95.4) (xy 148.6 95.4) (xy 148.6 97.8) (xy 147 97.8)
-				(xy 147 99.8) (xy 147 99.8) (xy 146 102) (xy 146 104.2)
+				(xy 147 99.8) (xy 146 102) (xy 146 104.2)
 			)
 		)
