File: PCB_files/Sprinkler_Controller_V2/Sprinkler_Controller_V2/Sprinkler_Controller_V2.kicad_sch (KiCad schematic)
At the start: 43 parts, among them J1 Screw_Terminal_01x02, J2 Screw_Terminal_01x11, SW1 SW_SPST, U1 ESP32_DevKit_V1_DOIT, U12 TPP362081-T6TR

Commit message: Changed capacitors
Parts:
- C1, C2: footprint Capacitor_THT:CP_Radial_D16.0mm_P7.50mm -> footprints:PCAP_12_5x25-THRU-ELECT_NCA
Changed lines of the file:
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@@
 	(label "Vin"
 		(at 60.96 22.86 0)
-		(fields_autoplaced yes)
 		(effects
 			(font
@@
 			)
 		)
-		(property "Footprint" "Capacitor_THT:CP_Radial_D16.0mm_P7.50mm"
+		(property "Footprint" "footprints:PCAP_12_5x25-THRU-ELECT_NCA"
 			(at 68.58 27.94 0)
 			(effects
@@
 			)
 		)
-		(property "Footprint" "Capacitor_THT:CP_Radial_D16.0mm_P7.50mm"
+		(property "Footprint" "footprints:PCAP_12_5x25-THRU-ELECT_NCA"
 			(at 60.96 27.94 0)
 			(effects
